File: hardware/solar/boost_regulator.kicad_sch (KiCad schematic)
At the start: 0 parts

Commit message: Design updates
Other:
- note added: "TBD"
Changed lines of the file:
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@@
 (kicad_sch (version 20211123) (generator eeschema)
   (paper "A4")
+  (title_block
+    (date "2022-01-20")
+    (rev "0.0.1")
+  )
   (wire (pts (xy 149.86 82.55) (xy 170.18 82.55))
     (stroke (width 0) (type default) (color 0 0 0 0))
   )
+  (text "TBD" (at 157.48 81.28 0)
+    (effects (font (size 1.27 1.27)) (justify left bottom))
+  )
   (hierarchical_label "5V0" (shape input) (at 170.18 82.55 0)
