File: hardware/solar/mcu.kicad_sch (KiCad schematic)
At the start: 0 parts

Commit message: Design updates
Other:
- note added: "TBD"
Changed lines of the file:
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@@
     (rev "0.0.1")
   )
+  (text "TBD" (at 115.57 86.36 0)
+    (effects (font (size 1.27 1.27)) (justify left bottom))
+  )
+  (hierarchical_label "CHARGE_CTL" (shape output) (at 96.52 90.17 0)
+    (effects (font (size 1.27 1.27)) (justify left))
+  )
+  (hierarchical_label "I2C" (shape bidirectional) (at 96.52 95.25 0)
+    (effects (font (size 1.27 1.27)) (justify left))
+  )
+  (hierarchical_label "VSENSE_SOLAR" (shape input) (at 96.52 85.09 0)
+    (effects (font (size 1.27 1.27)) (justify left))
+  )
+  (hierarchical_label "LOAD_SWITCH" (shape output) (at 96.52 92.71 0)
+    (effects (font (size 1.27 1.27)) (justify left))
+  )
+  (hierarchical_label "VSENSE_USB" (shape input) (at 96.52 82.55 0)
+    (effects (font (size 1.27 1.27)) (justify left))
+  )
+  (hierarchical_label "VSENSE_BAT" (shape input) (at 96.52 87.63 0)
+    (effects (font (size 1.27 1.27)) (justify left))
+  )
 )
