File: hardware/solar/solar-charger.kicad_sch (KiCad schematic)
At the start: 11 parts

Commit message: Design updates
Parts:
- removed D?: SB5200TA, symbol Device:D_Schottky
- removed J?: ISENSE_CHARGE, symbol Connector:Conn_01x02_Male
- added D? (x2): LED, symbol Device:LED
- added Q? (x2): AOI21357, symbol Device:Q_PMOS_GDS
- added R?: 100k, symbol Device:R_US
Connections:
- net GND: now also D?.1 (K), D?.1 (K), Q?.1 (G)
- net VSENSE_SOLAR: now also D?.2 (A)
- net VSENSE_USB: now also D?.2 (A), Q?.2 (D); no longer J?.2 (Pin_2)
- net INA219 (Current Sense)/I_IN: now reaches Q?.2 (D)
- net at J?.2 (Pin_2), Q?.1 (G), Q?.3 (S)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: now also Q?.3 (S)
- new net: J?.2 (Pin_2), Q?.2 (D), Q?.3 (S), R?.1
- new net LOAD_SWITCH: Q?.1 (G), R?.2
Other:
- sheet boost_regulator renamed Boost Regulator
- added sheet INA219 (Current Sense) (ina219.kicad_sch)
- sheet MCU ports: added CHARGE_CTL, I2C, LOAD_SWITCH, VSENSE_BAT, VSENSE_SOLAR, VSENSE_USB; removed none
- note added: ""Power Path" ->"
- note added: "<- Battery Charging"
- note added: "Current Sense Point (Short if not used)"
- note added: "I2C address = 0x40"
- note added: "Solar Power Indicator"
- note added: "System Power Indicator"
- note added: "TODO: NTC Measurement Circuit"
- note added: "To Raspberry Pi board (5.0V nom)"
- note added: "Using an Arduino for the breadboarded circuit"
- note removed: "Current Sense Point (Shunt if not used)"
- note removed: "NTC Measurement Circuit?"
- note removed: "To Raspberry Pi board"
- title: MCU -> Solar Charger Breadboard
- moved on the sheet: BT?, J?, Q?, R?, TH?
